File: ProtoGuard.kicad_sch (KiCad schematic)
At the start: 6 parts, among them J1 Conn_02x05_Odd_Even, U1 STM32G030K6Tx

Commit message: .
Parts:
- added C3: 10n, Capacitor_SMD:C_1206_3216Metric, symbol Device:C_Small
- added C4, C5, C6: 10u, Capacitor_SMD:C_1206_3216Metric, symbol Device:C_Small
- added D1, D3: B5819W, Diode_SMD:D_SOD-123, symbol Device:D_Schottky_Small
- added D2: RED, LED_SMD:LED_0603_1608Metric, symbol Device:LED_Small
- added D4: BZT52C12, EasyEDA:SOD-123_L2.7-W1.6-LS3.7-RD-1, symbol EasyEDA:BZT52C12_C2891780
- added D5: BZT52C5V1, EasyEDA:SOD-123_L2.7-W1.6-LS3.7-RD, symbol EasyEDA:BZT52C5V1_C2827905
- added L1: 10u, Inductor_SMD:L_Sunlord_MWSA1204S-100, symbol Device:L_Small
- added OLED1: X087-2832TSWIG02-H14, EasyEDA:OLED-SMD_X087-2832TSWIG02-H14, symbol EasyEDA:X087-2832TSWIG02-H14
- added Q1: AO4407A, EasyEDA:SOIC-8_L4.9-W3.9-P1.27-LS6.0-BL, symbol EasyEDA:AO4407A
- added R3: 47k, Resistor_SMD:R_0603_1608Metric, symbol Device:R_Small
- added R4: 15k, Resistor_SMD:R_0603_1608Metric, symbol Device:R_Small
- added R5: 270, Resistor_SMD:R_0603_1608Metric, symbol Device:R_Small
- added R6: 1k, Resistor_SMD:R_0201_0603Metric, symbol Device:R_Small
- added R7: 10k, Resistor_SMD:R_0603_1608Metric, symbol Device:R_Small
- added R8: 100k, Resistor_SMD:R_0603_1608Metric, symbol Device:R_Small
- added U2: (no value), Package_TO_SOT_SMD:TSOT-23-6, symbol MyLibrary:MP2359
- added U3: INA226, Package_SO:TSSOP-10_3x3mm_P0.5mm, symbol Sensor_Energy:INA226
- added U4: TPS2596xx, Package_SO:TI_SO-PowerPAD-8_ThermalVias, symbol Power_Management:TPS2596xx
- added U5: CH340N, Package_SO:JEITA_SOIC-8_3.9x4.9mm_P1.27mm, symbol Interface_USB:CH340N
- C2: value 4u7 -> 100n
Connections:
- net +3.3V: now also C4.1, C5.1, D2.2 (A), L1.2, R3.1
- net GND: now also C4.2, C5.2, C6.2, D1.2 (A), D5.2 (A), R5.2, R6.2, R7.2, U2.2 (GND)
- net I2C1_SDA: now reaches U1.1 (PB9)
- net ADC1_IN9: now reaches U1.16 (PB1)
- new net: R4.2, R5.1
- new net: D4.2 (A), Q1.4 (G), R7.1
- new net: U4.1 (GND), U4.9 (GND)
- new net: D2.1 (K), R6.1
- new net BUCK_BST: C3.1, U2.1 (BST)
- new net BUCK_EN: D5.1 (K), R8.2, U2.4 (EN)
- new net BUCK_FB: R3.2, R4.1, U2.3 (FB)
- new net BUCK_IN: C6.1, D3.1 (K), D4.1 (K), Q1.1 (S), Q1.2 (S), Q1.3 (S), R8.1, U2.5 (IN)
- new net BUCK_SW: C3.2, D1.1 (K), L1.1, U2.6 (SW)
- new net Vin_TERMINAL: Q1.5 (D), Q1.6 (D), Q1.7 (D), Q1.8 (D)
- new net Vin_USB: D3.2 (A)
- no-connect marks 3 -> 22
Other:
- note added: "MCU"
- note added: "PSU"
- moved on the sheet: C1, C2, J1, R1, R2, U1

Commit message: .
Parts:
- added C10, C12: 0.1u, Package_SO:SOIC-8_3.9x4.9mm_P1.27mm, symbol Device:C_Small
- added C11, C9: 4u7, Package_SO:SOIC-8_3.9x4.9mm_P1.27mm, symbol Device:C_Small
- added C7, C8: 1u, Capacitor_SMD:C_1206_3216Metric, symbol Device:C_Small
- added R9: 560k, Resistor_SMD:R_0603_1608Metric, symbol Device:R_Small
Connections:
- net +3.3V: now also OLED1.5 (VBAT), OLED1.8 (VDD), C10.1, C9.1
- net GND: now also OLED1.7 (VSS), C10.2, C11.2, C12.2, C9.2, R9.2
- net I2C2_SCL: now also OLED1.10 (SCL)
- net I2C2_SDA: now also OLED1.11 (SDA)
- net C2P: now reaches OLED1.1 (C2P)
- net C2P: now also C7.2
- net IREF: now reaches OLED1.12 (IREF)
- net IREF: now also R9.1
- net VCOMH: now reaches OLED1.13 (VCOMH)
- net VCC: now reaches OLED1.14 (VCC)
- net VCC: now also C11.1, C12.1
- net C2N: now reaches OLED1.2 (C2N)
- net C2N: now also C7.1
- net C1P: now reaches OLED1.3 (C1P)
- net C1P: now also C8.2
- net C1N: now reaches OLED1.4 (C1N)
- net C1N: now also C8.1
- net RES: now reaches OLED1.9 (~{RES})
- no-connect marks 22 -> 23
Other:
- note added: "PROVERI OVO"
- moved on the sheet: OLED1, U3, U4, U5

Commit message: .
Parts:
- added C13: 2u2, Package_SO:SOIC-8_3.9x4.9mm_P1.27mm, symbol Device:C_Small
- added C14: 100n, Package_SO:SOIC-8_3.9x4.9mm_P1.27mm, symbol Device:C_Small
- added C15: 4u7, Capacitor_SMD:C_1206_3216Metric, symbol Device:C_Small
- added C16: 4u7, Package_SO:SOIC-8_3.9x4.9mm_P1.27mm, symbol Device:C_Small
- added C17: 10u, Capacitor_SMD:C_1206_3216Metric, symbol Device:C_Small
- added L2: 4u7, Inductor_SMD:L_Sunlord_MWSA1204S-100, symbol Device:L_Small
- added Q2: FDN335N, EasyEDA:SOT-23-3_L3.0-W1.7-P0.95-LS2.9-BR, symbol EasyEDA:FDN335N
- added Q3: FDN338P, EasyEDA:SOT-23-3_L2.9-W1.6-P1.90-LS2.8-BR, symbol EasyEDA:FDN338P
- added R10, R11: 47k, Resistor_THT:R_Array_SIP4, symbol Device:R_Small
- added R12: 100k, Resistor_THT:R_Array_SIP4, symbol Device:R_Small
- added R13: 309k, Resistor_SMD:R_0201_0603Metric, symbol Device:R_Small
- added R14: 665k, Resistor_SMD:R_0201_0603Metric, symbol Device:R_Small
- added SW1: SW_Push, Package_DIP:DIP-8_W7.62mm, symbol Switch:SW_Push
- added U6: MCP1640Bx-xCHY, Package_TO_SOT_SMD:SOT-23-6, symbol Regulator_Switching:MCP1640Bx-xCHY
- C10, C12: value 0.1u -> 100n
- R1, R2: value 2k2 -> 4k7
Connections:
- net RES is gone; now on net SCREEN_RESET: OLED1.9 (~{RES})
- net +3.3V: now also C15.1, L2.1, U6.3 (EN), U6.6 (V_{IN}); no longer OLED1.5 (VBAT)
- net GND: now also C13.2, C14.2, C15.2, C16.2, C17.2, Q2.2 (S), R11.1, R12.1, R13.2, SW1.2, U6.2 (GND)
- net NRST: now also C14.1, SW1.1
- net VCOMH: now also C13.1
- net SCREEN_RESET: now reaches U1.18 (PA8)
- net SCREEN_RESET: now also R12.2
- net I2C1_SDA renamed SCREEN
- net SCREEN: now also Q2.1 (G), R11.2
- new net: Q2.3 (D), Q3.1 (G), R10.2
- new net +3V8: C17.1, Q3.2 (S), R10.1, R14.1, U6.5 (V_{OUT})
- new net BOOST_SW: L2.2, U6.1 (SW)
- new net BOOST_VFB: R13.1, R14.2, U6.4 (V_{FB})
- new net VBAT: C16.1, OLED1.5 (VBAT), Q3.3 (D)
- no-connect marks 23 -> 22
Other:
- note added: "BOOST"
- note added: "DISPLAY"
- note added: "DRUGI TRANZISTORI"
- note removed: "PROVERI OVO"
- moved on the sheet: C1, C10, C11, C12, C2, C7, C8, C9, J1, OLED1, R1, R2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

Commit message: .
Parts:
- added C18, C19: 100n, Package_SO:SOIC-8_3.9x4.9mm_P1.27mm, symbol Device:C_Small
- added D6: RED, LED_SMD:LED_0603_1608Metric, symbol Device:LED_Small
- added R15: 1k2, Resistor_SMD:R_0201_0603Metric, symbol Device:R_Small
Connections:
- net +3.3V: now also U5.5 (VCC), U5.8 (V3), C18.1, C19.1
- net +3V8: now also D6.2 (A)
- net GND: now also U5.3 (GND), C18.2, C19.2, R15.2
- net USART2_RX: now also U5.6 (TXD)
- net USART2_TX: now also U5.7 (RXD)
- net USB+: now reaches U5.1 (UD+)
- net USB-: now reaches U5.2 (UD-)
- new net: D6.1 (K), R15.1
- no-connect marks 22 -> 23
Other:
- moved on the sheet: C15, C17, L2, R13, R14, U5, U6

Commit message: .
Parts:
- added C20: 4n7, Package_SO:SOIC-8_3.9x4.9mm_P1.27mm, symbol Device:C_Small
- added J2: USB_C_Receptacle_USB2.0_14P, Package_SO:SOIC-16_3.9x9.9mm_P1.27mm, symbol Connector:USB_C_Receptacle_USB2.0_14P
- added R16, R17: 5k1, Resistor_THT:R_Array_SIP4, symbol Device:R_Small
- added R18: 1M, Resistor_THT:R_Array_SIP4, symbol Device:R_Small
- added U7: USBLC6-2SC6, Package_TO_SOT_SMD:SOT-23-6, symbol Power_Protection:USBLC6-2SC6
Connections:
- net +3.3V: now also U7.5 (VBUS)
- net GND: now also C20.2, J2.A1 (GND), J2.A12 (GND), J2.B1 (GND), J2.B12 (GND), R16.2, R17.2, R18.2, U7.2 (GND)
- net USB+: now also J2.A6 (D+), J2.B6 (D+), U7.1 (I/O1), U7.6 (I/O1)
- net USB-: now also J2.A7 (D-), J2.B7 (D-), U7.3 (I/O2), U7.4 (I/O2)
- net Vin_USB: now also J2.A4 (VBUS), J2.A9 (VBUS), J2.B4 (VBUS), J2.B9 (VBUS)
- new net: J2.A5 (CC1), R17.1
- new net: J2.B5 (CC2), R16.1
- new net SH: C20.1, J2.SH (SHIELD), R18.1
Other:
- note added: "BOOST 3V8"
- note added: "USB"
- note added: "USB TO UART"
- note removed: "BOOST"
- note removed: "DRUGI TRANZISTORI"
- moved on the sheet: C18, C19, U5

Commit message: .
Parts:
- added C21: 100n, Package_SO:SOIC-8_3.9x4.9mm_P1.27mm, symbol Device:C_Small
- added J3: Screw_Terminal_01x02, symbol Connector:Screw_Terminal_01x02
- added R19: (no value), Resistor_THT:R_Array_SIP4, symbol Device:R_Small
Connections:
- net +3.3V: now also U3.6 (VS), C21.1
- net GND: now also U3.1 (A1), U3.2 (A0), U3.7 (GND), C21.2, J3.2 (Pin_2)
- net I2C2_SCL: now also U3.5 (SCL)
- net I2C2_SDA: now also U3.4 (SDA)
- net Vin_TERMINAL: now also J3.1 (Pin_1)
- net VSHUNT+: now reaches U3.10 (Vin+)
- net ALERT: now reaches U3.3 (~{Alert})
- net VSHUNT-: now reaches U3.8 (Vbus)
- net VSHUNT-: now also U3.9 (Vin-)
Other:
- note added: "INPUT"
- note removed: "USB"
- moved on the sheet: C20, R18, U3, U7

Commit message: .
Parts:
- added R20: 10k, Resistor_THT:R_Array_SIP4, symbol Device:R_Small
- added RV1: 10k, Package_SO:TSSOP-20_4.4x6.5mm_P0.65mm, symbol Device:R_Potentiometer_Small
- R19: value (none) -> 20m
Connections:
- net VSHUNT+ is gone; now on net BUCK_IN: U3.10 (Vin+)
- net VSHUNT- is gone; now on net VOUT: U3.8 (Vbus), U3.9 (Vin-)
- net +3.3V: now also R20.1, RV1.1
- net ADC1_IN9: now also RV1.2
- net ALERT: now also R20.2
- net BUCK_IN: now also R19.1
- net GND: now also RV1.3
- net VOUT: now reaches R19.2

Commit message: .
Parts:
- removed U4: TPS2596xx, Package_SO:TI_SO-PowerPAD-8_ThermalVias, symbol Power_Management:TPS2596xx
- added C13, C22, C4: 100n, Package_SO:SOIC-8_3.9x4.9mm_P1.27mm, symbol Device:C_Small
- added C21: 3n3, Capacitor_SMD:C_1206_3216Metric, symbol Device:C_Small
- added C26: 1u, Capacitor_SMD:C_1206_3216Metric, symbol Device:C_Small
- added D5: SS34, Diode_SMD:D_SMA, symbol Diode:SS34
- added J4: Screw_Terminal_01x02, symbol Connector:Screw_Terminal_01x02
- added R14, R16, R18: 10, Resistor_THT:R_Array_SIP4, symbol Device:R_Small
- added R19: 10k, Resistor_THT:R_Array_SIP4, symbol Device:R_Small
- added R24: 499, Resistor_THT:R_Array_SIP4, symbol Device:R_Small
- added SW2: SW_Push, Package_DIP:DIP-8_W7.62mm, symbol Switch:SW_Push
- added U7: TPS259570DSGR, EasyEDA:WDFN-8_L2.0-W2.0-P0.50-BL-EP, symbol EasyEDA:TPS259570DSGR
- R15: renamed from R19; value 20m -> 22m
- R20: value 10k -> 100k
- renumbered C6 to C1, C21 to C10, C4 to C11, C5 to C12, C16 to C14, C7 to C15, C9 to C16, C10 to C17, C8 to C18, C17 to C19, C18 to C2, C13 to C20, C11 to C23, C12 to C24, C15 to C25, C19 to C3, C20 to C5, C14 to C6, C1 to C7, C2 to C8, C3 to C9, D4 to D1, D3 to D2, D5 to D3, D1 to D4, D2 to D6, D6 to D7, J2 to J1, J1 to J2, R7 to R1, R4 to R10, R5 to R11, R11 to R12, R10 to R13, R6 to R17, R16 to R2, R9 to R21, R14 to R22, R13 to R23, R15 to R25, R17 to R3, R18 to R4, R1 to R5, R2 to R6, R8 to R7, R12 to R8, R3 to R9, U5 to U1, U1 to U2, U7 to U3, U2 to U4, U3 to U5
Connections:
- net +3.3V: no longer R20.1
- net ADC1_IN9: now also C4.1
- net ALERT: now also R20.1, U2.13 (PA6), R19.2, U7.2 (EN/UVLO); no longer R20.2
- net BUCK_IN: now also C22.1, U7.3 (IN), U7.4 (IN); no longer R15.1, U5.10 (Vin+)
- net GND: now also R20.2, C21.1, C22.2, C26.2, C4.2, D5.2 (A), J4.2 (Pin_2), R24.2, SW2.2, U7.8 (GND), U7.9 (GND)
- net VOUT: now also D5.1 (K), J4.1 (Pin_1), R16.2, R18.1; no longer U5.8 (Vbus), U5.9 (Vin-)
- net OUTPUT_EN: now reaches U2.12 (PA5)
- net OUTPUT_EN: now also R19.1
- net REARM: now reaches U2.17 (PB2)
- net REARM: now also SW2.1
- new net: C21.2, U7.1 (dVdt)
- new net: R24.1, U7.7 (ILM)
- new net TPS_OUT: C26.1, R14.2, R15.1, U7.5 (OUT)
- new net VBUS_INA226V: R18.2, U5.8 (Vbus)
- new net VSHUNT+: C13.1, R14.1, U5.10 (Vin+)
- new net VSHUNT-: C13.2, R16.1, U5.9 (Vin-)
- no-connect marks 23 -> 21
Other:
- note added: "MEASUREMENT"
- note added: "PROTECTION LOGIC"
- moved on the sheet: C10, C6, C7, C8, J2, R15, R5, R6, RV1, SW1, U5
