File: ProtoGuard.kicad_sch (KiCad schematic)
At the start: 78 parts, among them J1 USB_C_Receptacle_USB2.0_14P, J2 Conn_02x05_Odd_Even, J3 Screw_Terminal_01x02, J4 Screw_Terminal_01x02, Q1 AO4407A, Q2 FDN335N, Q3 FDN338P, SW1 SW_Push, SW2 SW_Push, U1 CH340N, U2 STM32G030K6Tx, U3 USBLC6-2SC6, U5 INA226, U6 MCP1640Bx-xCHY, U7 TPS259570DSGR

Commit message: .
Parts:
- removed J1: USB_C_Receptacle_USB2.0_14P, Package_SO:SOIC-16_3.9x9.9mm_P1.27mm, symbol Connector:USB_C_Receptacle_USB2.0_14P
- removed L1: 10u, Inductor_SMD:L_Sunlord_MWSA1204S-100, symbol Device:L_Small
- removed L2: 4u7, Inductor_SMD:L_Sunlord_MWSA1204S-100, symbol Device:L_Small
- added C29: 47u, Capacitor_SMD:CP_Elec_6.3x7.7, symbol Device:C_Polarized_Small_US
- added D8: B5819W, Diode_SMD:D_SOD-123, symbol Device:D_Schottky_Small
- added J5: USB_C_Receptacle_USB2.0_16P, Connector_USB:USB_C_Receptacle_HRO_TYPE-C-31-M-12, symbol Connector:USB_C_Receptacle_USB2.0_16P
- added L1: FNR3015S4R7MT, EasyEDA:IND-SMD_L3.0-W3.0_FNR30XXS, symbol EasyEDA:FNR3015S4R7MT
- added L3: SMNR4030-100MT, EasyEDA:IND-SMD_L4.0-W4.0_SMNR4030, symbol EasyEDA:SMNR4030-100MT
- C1: LCSC (none) -> C13585; LCSC Part # C13585 -> (none)
- C10, C13, C17, C2, C24, C3, C4, C6, C8: footprint Package_SO:SOIC-8_3.9x4.9mm_P1.27mm -> Capacitor_SMD:C_0402_1005Metric; LCSC (none) -> C307331
- C11, C12, C19: footprint Capacitor_SMD:C_1206_3216Metric -> Capacitor_SMD:C_0805_2012Metric; LCSC (none) -> C15850; LCSC Part # C13585 -> (none)
- C14, C16, C23, C7: footprint Package_SO:SOIC-8_3.9x4.9mm_P1.27mm -> Capacitor_SMD:C_0805_2012Metric; LCSC (none) -> C1779
- C15, C18, C26: footprint Capacitor_SMD:C_1206_3216Metric -> Capacitor_SMD:C_0603_1608Metric; LCSC (none) -> C15849; LCSC Part # C13585 -> (none)
- C20: footprint Package_SO:SOIC-8_3.9x4.9mm_P1.27mm -> Capacitor_SMD:C_0805_2012Metric; LCSC (none) -> C19110
- C21: footprint Capacitor_SMD:C_1206_3216Metric -> Capacitor_SMD:C_0402_1005Metric; LCSC (none) -> C1536; LCSC Part # C13585 -> (none)
- C22: footprint Package_SO:SOIC-8_3.9x4.9mm_P1.27mm -> Capacitor_SMD:C_0603_1608Metric; LCSC (none) -> C1591
- C25: footprint Capacitor_SMD:C_1206_3216Metric -> Capacitor_SMD:C_0805_2012Metric; LCSC (none) -> C1779
- C5: footprint Package_SO:SOIC-8_3.9x4.9mm_P1.27mm -> Capacitor_SMD:C_0603_1608Metric; LCSC (none) -> C53987
- C9: footprint Capacitor_SMD:C_1206_3216Metric -> Capacitor_SMD:C_0402_1005Metric; LCSC (none) -> C15195; LCSC Part # C1846 -> (none)
- D1: LCSC (none) -> C2891780; LCSC Part C2891780 -> (none)
- D2, D4: LCSC (none) -> C9900270134; LCSC Part # C9900270134 -> (none)
- D3: LCSC (none) -> C2827905; LCSC Part C2827905 -> (none)
- J3: footprint (none) -> TerminalBlock_Phoenix:TerminalBlock_Phoenix_MKDS-1,5-2-5.08_1x02_P5.08mm_Horizontal
- J4: footprint (none) -> TerminalBlock_Philmore:TerminalBlock_Philmore_TB132_1x02_P5.00mm_Horizontal
- OLED1: LCSC (none) -> C18723015; LCSC Part C18723015 -> (none)
- Q1: LCSC (none) -> C16072; LCSC Part C16072 -> (none)
- Q2: LCSC (none) -> C241804; LCSC Part C241804 -> (none)
- Q3: LCSC (none) -> C24855; LCSC Part C24855 -> (none)
- R1: footprint Resistor_SMD:R_0603_1608Metric -> Resistor_SMD:R_0402_1005Metric; LCSC (none) -> C25744
- R10: footprint Resistor_SMD:R_0603_1608Metric -> Resistor_SMD:R_0402_1005Metric; LCSC (none) -> C25756; LCSC Part # C22809 -> (none)
- R11: footprint Resistor_SMD:R_0603_1608Metric -> Resistor_SMD:R_0402_1005Metric; LCSC (none) -> C22966; LCSC Part # C22966 -> (none)
- R12, R13: footprint Resistor_THT:R_Array_SIP4 -> Resistor_SMD:R_0402_1005Metric; LCSC (none) -> C25792
- R14, R16, R18: footprint Resistor_THT:R_Array_SIP4 -> Resistor_SMD:R_0402_1005Metric; LCSC (none) -> C25077
- R15: footprint Resistor_THT:R_Array_SIP4 -> Resistor_SMD:R_2512_6332Metric; LCSC (none) -> C2994626
- R17: footprint Resistor_SMD:R_0201_0603Metric -> Resistor_SMD:R_0402_1005Metric; LCSC (none) -> C11702; LCSC Part # C21190 -> (none)
- R19: footprint Resistor_THT:R_Array_SIP4 -> Resistor_SMD:R_0402_1005Metric; LCSC (none) -> C25744
- R2, R3: footprint Resistor_THT:R_Array_SIP4 -> Resistor_SMD:R_0402_1005Metric; LCSC (none) -> C25905
- R20, R8: footprint Resistor_THT:R_Array_SIP4 -> Resistor_SMD:R_0402_1005Metric; LCSC (none) -> C25741
- R21: footprint Resistor_SMD:R_0603_1608Metric -> Resistor_SMD:R_0402_1005Metric; LCSC (none) -> C132339; LCSC Part # C22809 -> (none)
- R22: footprint Resistor_SMD:R_0201_0603Metric -> Resistor_SMD:R_0402_1005Metric; LCSC (none) -> C56583; LCSC Part # C21190 -> (none)
- R23: footprint Resistor_SMD:R_0201_0603Metric -> Resistor_SMD:R_0402_1005Metric; LCSC (none) -> C21190; LCSC Part # C21190 -> (none)
- R24: footprint Resistor_THT:R_Array_SIP4 -> Resistor_SMD:R_0402_1005Metric; LCSC (none) -> C4125
- R25: footprint Resistor_SMD:R_0201_0603Metric -> Resistor_SMD:R_0402_1005Metric; LCSC (none) -> C25862; LCSC Part # C21190 -> (none)
- R4: footprint Resistor_THT:R_Array_SIP4 -> Resistor_SMD:R_0603_1608Metric
- R5, R6: footprint Resistor_THT:R_Array_SIP4 -> Resistor_SMD:R_0402_1005Metric; LCSC (none) -> C25900
- R7: footprint Resistor_SMD:R_0603_1608Metric -> Resistor_SMD:R_0402_1005Metric; LCSC (none) -> C25741
- R9: footprint Resistor_SMD:R_0603_1608Metric -> Resistor_SMD:R_0402_1005Metric; LCSC (none) -> C25792
- RV1: footprint Package_SO:TSSOP-20_4.4x6.5mm_P0.65mm -> Potentiometer_THT:Potentiometer_Alps_RK09K_Single_Vertical
- SW1, SW2: footprint Package_DIP:DIP-8_W7.62mm -> Button_Switch_SMD:SW_SPST_TL3342
- U4: LCSC (none) -> C14259; LCSC Part # C14259 -> (none)
- U7: LCSC (none) -> C1849463; LCSC Part C1849463 -> (none)
Connections:
- net +3.3V: now also L1.1, L3.2
- net BOOST_SW: now also L1.2
- net BUCK_IN: now also D8.1 (K); no longer C22.1, D1.1 (K), Q1.1 (S), Q1.2 (S), Q1.3 (S), U7.3 (IN), U7.4 (IN)
- net BUCK_SW: now also L3.1
- net GND: now also C29.2, J5.A1 (GND), J5.A12 (GND), J5.B1 (GND), J5.B12 (GND)
- net SH: now also J5.SH (SHIELD)
- net USB+: now also J5.A6 (D+), J5.B6 (D+)
- net USB-: now also J5.A7 (D-), J5.B7 (D-)
- net Vin_USB: now also J5.A4 (VBUS), J5.A9 (VBUS), J5.B4 (VBUS), J5.B9 (VBUS)
- net at R3.1: now also J5.A5 (CC1)
- net at R2.1: now also J5.B5 (CC2)
- new net TERMINAL_PROT: C22.1, C29.1, D1.1 (K), D8.2 (A), Q1.1 (S), Q1.2 (S), Q1.3 (S), U7.3 (IN), U7.4 (IN)
- no-connect marks 21 -> 23
Other:
- moved on the sheet: C1, C11, C12, C21, C22, C26, C9, D1, D2, D3, D4, D6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

Commit message: .
Parts:
- C25: LCSC Part # C13585 -> (none)
- D2, D4, D8: LCSC C9900270134 -> (none)
- R1, R7, R9: LCSC Part # C25819 -> (none)
- R11: LCSC C22966 -> (none)
- R23: LCSC C21190 -> (none)
